File: WindowOpener/WindowOpener.kicad_sch (KiCad schematic)
At the start: 32 parts, among them J1 Conn_ST_STDC14, J2 UEXT_Host, SW1 SW_Push, SW2 SW_SPDT_XKB, U1 STM32L152RCTxA, U2 AM2302, Y1 8MHz, Y2 32.768kHz

Commit message: Power hozzáadva
Other:
- sheet Power+USB renamed Power
Changed lines of the file:
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@@
 			(color 0 0 0 0.0000)
 		)
-		(property "Sheetname" "Power+USB"
+		(property "Sheetname" "Power"
 			(at 148.59 137.7184 0)
 			(effects

Commit message: v0.1
Other:
- sheet Power renamed MCU+Motors Power
Changed lines of the file:
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@@
 		)
 		(instances
-			(project "Aramkortervezes_projekt"
+			(project "WindowOpener"
 				(path "/9cc66d3b-a4f0-4570-ad5d-091fde92d938"
 					(reference "Y1")
@@
 		)
 		(instances
-			(project "Aramkortervezes_projekt"
+			(project "WindowOpener"
 				(path "/9cc66d3b-a4f0-4570-ad5d-091fde92d938"
 					(reference "#PWR014")
@@
 		)
 		(instances
-			(project "Aramkortervezes_projekt"
+			(project "WindowOpener"
 				(path "/9cc66d3b-a4f0-4570-ad5d-091fde92d938"
 					(reference "FB1")
@@
 		)
 		(instances
-			(project "Aramkortervezes_projekt"
+			(project "WindowOpener"
 				(path "/9cc66d3b-a4f0-4570-ad5d-091fde92d938"
 					(reference "R8")
@@
 		)
 		(instances
-			(project "Aramkortervezes_projekt"
+			(project "WindowOpener"
 				(path "/9cc66d3b-a4f0-4570-ad5d-091fde92d938"
 					(reference "R21")
@@
 		)
 		(instances
-			(project "Aramkortervezes_projekt"
+			(project "WindowOpener"
 				(path "/9cc66d3b-a4f0-4570-ad5d-091fde92d938"
 					(reference "R2")
@@
 		)
 		(instances
-			(project "Aramkortervezes_projekt"
+			(project "WindowOpener"
 				(path "/9cc66d3b-a4f0-4570-ad5d-091fde92d938"
 					(reference "#PWR01")
@@
 		)
 		(instances
-			(project "Aramkortervezes_projekt"
+			(project "WindowOpener"
 				(path "/9cc66d3b-a4f0-4570-ad5d-091fde92d938"
 					(reference "C10")
@@
 		)
 		(instances
-			(project "Aramkortervezes_projekt"
+			(project "WindowOpener"
 				(path "/9cc66d3b-a4f0-4570-ad5d-091fde92d938"
 					(reference "R1")
@@
 		)
 		(instances
-			(project ""
+			(project "WindowOpener"
 				(path "/9cc66d3b-a4f0-4570-ad5d-091fde92d938"
 					(reference "U2")
@@
 		)
 		(instances
-			(project "Aramkortervezes_projekt"
+			(project "WindowOpener"
 				(path "/9cc66d3b-a4f0-4570-ad5d-091fde92d938"
 					(reference "U1")
@@
 		)
 		(instances
-			(project "Aramkortervezes_projekt"
+			(project "WindowOpener"
 				(path "/9cc66d3b-a4f0-4570-ad5d-091fde92d938"
 					(reference "C6")
@@
 		)
 		(instances
-			(project "Aramkortervezes_projekt"
+			(project "WindowOpener"
 				(path "/9cc66d3b-a4f0-4570-ad5d-091fde92d938"
 					(reference "R3")
@@
 		)
 		(instances
-			(project "Aramkortervezes_projekt"
+			(project "WindowOpener"
 				(path "/9cc66d3b-a4f0-4570-ad5d-091fde92d938"
 					(reference "C5")
@@
 		)
 		(instances
-			(project "Aramkortervezes_projekt"
+			(project "WindowOpener"
 				(path "/9cc66d3b-a4f0-4570-ad5d-091fde92d938"
 					(reference "#PWR04")
@@
 		)
 		(instances
-			(project "Aramkortervezes_projekt"
+			(project "WindowOpener"
 				(path "/9cc66d3b-a4f0-4570-ad5d-091fde92d938"
 					(reference "#PWR08")
@@
 		)
 		(instances
-			(project "Aramkortervezes_projekt"
+			(project "WindowOpener"
 				(path "/9cc66d3b-a4f0-4570-ad5d-091fde92d938"
 					(reference "R5")
@@
 		)
 		(instances
-			(project "Aramkortervezes_projekt"
+			(project "WindowOpener"
 				(path "/9cc66d3b-a4f0-4570-ad5d-091fde92d938"
 					(reference "#PWR012")
@@
 		)
 		(instances
-			(project "Aramkortervezes_projekt"
+			(project "WindowOpener"
 				(path "/9cc66d3b-a4f0-4570-ad5d-091fde92d938"
 					(reference "#FLG03")
@@
 		)
 		(instances
-			(project "Aramkortervezes_projekt"
+			(project "WindowOpener"
 				(path "/9cc66d3b-a4f0-4570-ad5d-091fde92d938"
 					(reference "#PWR06")
@@
 		)
 		(instances
-			(project "Aramkortervezes_projekt"
+			(project "WindowOpener"
 				(path "/9cc66d3b-a4f0-4570-ad5d-091fde92d938"
 					(reference "#PWR02")
@@
 		)
 		(instances
-			(project "Aramkortervezes_projekt"
+			(project "WindowOpener"
 				(path "/9cc66d3b-a4f0-4570-ad5d-091fde92d938"
 					(reference "#PWR020")
@@
 		)
 		(instances
-			(project ""
+			(project "WindowOpener"
 				(path "/9cc66d3b-a4f0-4570-ad5d-091fde92d938"
 					(reference "J2")
@@
 		)
 		(instances
-			(project "Aramkortervezes_projekt"
+			(project "WindowOpener"
 				(path "/9cc66d3b-a4f0-4570-ad5d-091fde92d938"
 					(reference "C12")
@@
 		)
 		(instances
-			(project "Aramkortervezes_projekt"
+			(project "WindowOpener"
 				(path "/9cc66d3b-a4f0-4570-ad5d-091fde92d938"
 					(reference "#PWR021")
@@
 		)
 		(instances
-			(project ""
+			(project "WindowOpener"
 				(path "/9cc66d3b-a4f0-4570-ad5d-091fde92d938"
 					(reference "SW2")
@@
 		)
 		(instances
-			(project "Aramkortervezes_projekt"
+			(project "WindowOpener"
 				(path "/9cc66d3b-a4f0-4570-ad5d-091fde92d938"
 					(reference "R7")
@@
 		)
 		(instances
-			(project "Aramkortervezes_projekt"
+			(project "WindowOpener"
 				(path "/9cc66d3b-a4f0-4570-ad5d-091fde92d938"
 					(reference "#PWR03")
@@
 		)
 		(instances
-			(project ""
+			(project "WindowOpener"
 				(path "/9cc66d3b-a4f0-4570-ad5d-091fde92d938"
 					(reference "SW1")
@@
 		)
 		(instances
-			(project "Aramkortervezes_projekt"
+			(project "WindowOpener"
 				(path "/9cc66d3b-a4f0-4570-ad5d-091fde92d938"
 					(reference "C1")
@@
 		)
 		(instances
-			(project "Aramkortervezes_projekt"
+			(project "WindowOpener"
 				(path "/9cc66d3b-a4f0-4570-ad5d-091fde92d938"
 					(reference "C4")
@@
 		)
 		(instances
-			(project "Aramkortervezes_projekt"
+			(project "WindowOpener"
 				(path "/9cc66d3b-a4f0-4570-ad5d-091fde92d938"
 					(reference "C3")
@@
 		)
 		(instances
-			(project "Aramkortervezes_projekt"
+			(project "WindowOpener"
 				(path "/9cc66d3b-a4f0-4570-ad5d-091fde92d938"
 					(reference "C9")
@@
 		)
 		(instances
-			(project "Aramkortervezes_projekt"
+			(project "WindowOpener"
 				(path "/9cc66d3b-a4f0-4570-ad5d-091fde92d938"
 					(reference "#PWR011")
@@
 		)
 		(instances
-			(project "Aramkortervezes_projekt"
+			(project "WindowOpener"
 				(path "/9cc66d3b-a4f0-4570-ad5d-091fde92d938"
 					(reference "#PWR015")
@@
 		)
 		(instances
-			(project "Aramkortervezes_projekt"
+			(project "WindowOpener"
 				(path "/9cc66d3b-a4f0-4570-ad5d-091fde92d938"
 					(reference "#PWR013")
@@
 		)
 		(instances
-			(project "Aramkortervezes_projekt"
+			(project "WindowOpener"
 				(path "/9cc66d3b-a4f0-4570-ad5d-091fde92d938"
 					(reference "R22")
@@
 		)
 		(instances
-			(project "Aramkortervezes_projekt"
+			(project "WindowOpener"
 				(path "/9cc66d3b-a4f0-4570-ad5d-091fde92d938"
 					(reference "R6")
@@
 		)
 		(instances
-			(project "Aramkortervezes_projekt"
+			(project "WindowOpener"
 				(path "/9cc66d3b-a4f0-4570-ad5d-091fde92d938"
 					(reference "C2")
@@
 		)
 		(instances
-			(project "Aramkortervezes_projekt"
+			(project "WindowOpener"
 				(path "/9cc66d3b-a4f0-4570-ad5d-091fde92d938"
 					(reference "#PWR07")
@@
 		)
 		(instances
-			(project "Aramkortervezes_projekt"
+			(project "WindowOpener"
 				(path "/9cc66d3b-a4f0-4570-ad5d-091fde92d938"
 					(reference "R4")
@@
 		)
 		(instances
-			(project "Aramkortervezes_projekt"
+			(project "WindowOpener"
 				(path "/9cc66d3b-a4f0-4570-ad5d-091fde92d938"
 					(reference "C7")
@@
 		)
 		(instances
-			(project "Aramkortervezes_projekt"
+			(project "WindowOpener"
 				(path "/9cc66d3b-a4f0-4570-ad5d-091fde92d938"
 					(reference "#PWR010")
@@
 		)
 		(instances
-			(project "Aramkortervezes_projekt"
+			(project "WindowOpener"
 				(path "/9cc66d3b-a4f0-4570-ad5d-091fde92d938"
 					(reference "#PWR05")
@@
 		)
 		(instances
-			(project "Aramkortervezes_projekt"
+			(project "WindowOpener"
 				(path "/9cc66d3b-a4f0-4570-ad5d-091fde92d938"
 					(reference "J1")
@@
 		)
 		(instances
-			(project "Aramkortervezes_projekt"
+			(project "WindowOpener"
 				(path "/9cc66d3b-a4f0-4570-ad5d-091fde92d938"
 					(reference "C8")
@@
 		)
 		(instances
-			(project "Aramkortervezes_projekt"
+			(project "WindowOpener"
 				(path "/9cc66d3b-a4f0-4570-ad5d-091fde92d938"
 					(reference "R9")
@@
 		)
 		(instances
-			(project "Aramkortervezes_projekt"
+			(project "WindowOpener"
 				(path "/9cc66d3b-a4f0-4570-ad5d-091fde92d938"
 					(reference "#PWR09")
@@
 		)
 		(instances
-			(project "Aramkortervezes_projekt"
+			(project "WindowOpener"
 				(path "/9cc66d3b-a4f0-4570-ad5d-091fde92d938"
 					(reference "#FLG02")
@@
 		)
 		(instances
-			(project "Aramkortervezes_projekt"
+			(project "WindowOpener"
 				(path "/9cc66d3b-a4f0-4570-ad5d-091fde92d938"
 					(reference "Y2")
@@
 		)
 		(instances
-			(project "Aramkortervezes_projekt"
+			(project "WindowOpener"
 				(path "/9cc66d3b-a4f0-4570-ad5d-091fde92d938"
 					(reference "C11")
@@
 			(color 0 0 0 0.0000)
 		)
-		(property "Sheetname" "Power"
+		(property "Sheetname" "MCU+Motors Power"
 			(at 148.59 137.7184 0)
 			(effects

Commit message: v0.2
Parts:
- C6: footprint Capacitor_SMD:C_2220_5750Metric_Pad1.97x5.40mm_HandSolder -> Capacitor_SMD:C_1206_3216Metric_Pad1.33x1.80mm_HandSolder; Store link https://hu.farnell.com/chemi-con/kts500b106m55n0t00/cap-mlc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 -> https://hu.farnell.com/multicomp-pro/1206x106k160ct/cap-10-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
Other:
- sheet MCU+Motors Power ports: added IN1_1, IN1_2, IN2_1, IN2_2; removed none
Changed lines of the file:
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@@
 	(title_block
 		(title "SmartHome WindowOpener")
-		(date "2026-03-08")
+		(date "2026-03-21")
 	)
 	(rectangle
@@
 			)
 		)
-		(property "Footprint" "Capacitor_SMD:C_2220_5750Metric_Pad1.97x5.40mm_HandSolder"
+		(property "Footprint" "Capacitor_SMD:C_1206_3216Metric_Pad1.33x1.80mm_HandSolder"
 			(at 271.4752 40.64 0)
 			(effects
@@
 			)
 		)
-		(property "Datasheet" "https://www.farnell.com/datasheets/4451690.pdf"
+		(property "Datasheet" "https://hu.farnell.com/multicomp-pro/1206x106k160ct/cap-10-f-16v-10-x5r-1206/dp/2497151"
 			(at 270.51 36.83 0)
 			(effects
@@
 			)
 		)
-		(property "Store link" "https://hu.farnell.com/chemi-con/kts500b106m55n0t00/cap-mlcc-10uf-50vdc-x7r-2220/dp/4629786"
+		(property "Store link" "https://hu.farnell.com/multicomp-pro/1206x106k160ct/cap-10-f-16v-10-x5r-1206/dp/2497151"
 			(at 270.51 36.83 0)
 			(effects
@@
 			)
 		)
+		(pin "IN1_1" input
+			(at 148.59 140.97 180)
+			(effects
+				(font
+					(size 1.27 1.27)
+				)
+				(justify left)
+			)
+		)
+		(pin "IN2_1" input
+			(at 148.59 143.51 180)
+			(effects
+				(font
+					(size 1.27 1.27)
+				)
+				(justify left)
+			)
+		)
+		(pin "IN1_2" input
+			(at 148.59 146.05 180)
+			(effects
+				(font
+					(size 1.27 1.27)
+				)
+				(justify left)
+			)
+		)
+		(pin "IN2_2" input
+			(at 148.59 148.59 180)
+			(effects
+				(font
+					(size 1.27 1.27)
+				)
+				(justify left)
+			)
+		)

Commit message: v0.3
Parts:
- removed R5: 100R, Resistor_SMD:R_2010_5025Metric_Pad1.40x2.65mm_HandSolder, symbol Device:R
- removed U2: AM2302, Sensor:ASAIR_AM2302_P2.54mm_Vertical, symbol Sensor:AM2302
Connections:
- net ADC1: now reaches U1.15 (PA1)
- net ADC2: now reaches U1.16 (PA2)
- net ADC3: now reaches U1.20 (PA4)
- net ADC4: now reaches U1.21 (PA5)
- net ADC5: now reaches U1.24 (PC4)
- net IN2_1: now reaches U1.37 (PC6)
- net LED3: now reaches U1.38 (PC7)
- net LED4: now reaches U1.39 (PC8)
- net LED5: now reaches U1.40 (PC9)
- net IN1_1: now reaches U1.50 (PA15)
- net LED6: now reaches U1.51 (PC10)
- net LED7: now reaches U1.52 (PC11)
- net IN1_2: now reaches U1.61 (PB8)
- net IN2_2: now reaches U1.62 (PB9)
- net LED2: now reaches U1.9 (PC1)
- no-connect marks 41 -> 26
Other:
- sheet MCU+Motors Power renamed MCU+Motors power
- added sheet LEDs (leds.kicad_sch)
- added sheet Sensors (sensors.kicad_sch)
- sheet MCU+Motors power ports: added none; removed IN1_1, IN1_2, IN2_1, IN2_2
- note added: "MCU+Motors power"
- note added: "Power LEDs"
- note added: "Sensors"
- note removed: "Battery management"
- note removed: "DHT22 szenzor"
- moved on the sheet: J2, R21, R22, R9
