File: WindowOpener/power.kicad_sch (KiCad schematic)
At the start: 0 parts

Commit message: Power hozzáadva
Parts:
- added C13: 10uF, Capacitor_SMD:C_2220_5750Metric_Pad1.97x5.40mm_HandSolder, symbol Device:C
- added C14: 22uF, Capacitor_SMD:C_1206_3216Metric_Pad1.33x1.80mm_HandSolder, symbol Device:C
- added J3, J4: Conn_01x02, Battery:BatteryHolder_Keystone_1042_1x18650, symbol Connector_Generic:Conn_01x02
- added LED1: GREEN, SmartHomeFootprints:LED_1411, symbol Device:LED
- added R10: 15R, Resistor_SMD:R_1210_3225Metric_Pad1.30x2.65mm_HandSolder, symbol Device:R
- added R11: 20R, Resistor_SMD:R_1210_3225Metric_Pad1.30x2.65mm_HandSolder, symbol Device:R
- added U3: AZ1117CH2-3.3, Package_TO_SOT_SMD:SOT-223-3_TabPin2, symbol Regulator_Linear:AZ1117CH2-3.3
Connections:
- new net: R10.2, R11.1
- new net: LED1.2 (A), R11.2
- new net: J3.1 (Pin_1), J4.2 (Pin_2)
- new net: C13.1, J3.2 (Pin_2), U3.1 (IN)
- new net 3V3: C14.1, R10.1, U3.3 (OUT)
- new net GND: C13.2, C14.2, J4.1 (Pin_1), LED1.1 (K), U3.2 (GND)

Commit message: v0.1
Parts:
- J3: value Conn_01x02 -> Batt_Conn1
- J4: value Conn_01x02 -> Batt_Conn2
Other:
- note added: "MC tápellátás"
Changed lines of the file:
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@@
 		(date "2026-03-08")
+	)
+	(rectangle
+		(start 24.13 19.05)
+		(end 139.7 74.93)
+		(stroke
+			(width 0)
+			(type dash)
+		)
+		(fill
+			(type none)
+		)
+	)
+	(text "MC tápellátás"
+		(exclude_from_sim no)
+		(at 31.75 21.844 0)
+		(effects
+			(font
+				(size 1.27 1.27)
+			)
+		)
 	)
 	(junction
@@
 			)
 		)
-		(property "Value" "Conn_01x02"
+		(property "Value" "Batt_Conn1"
 			(at 37.846 39.37 0)
 			(effects
@@
 		)
 		(pin "2"
+			(alternate "Negative")
 		)
 		(pin "1"
+			(alternate "Positve")
 		)
 		(instances
@@
 	)
 	(symbol
+		(lib_name "Conn_01x02_1")
 		(lib_id "Connector_Generic:Conn_01x02")
 		(at 45.72 48.26 180)
@@
 			)
 		)
-		(property "Value" "Conn_01x02"
+		(property "Value" "Batt_Conn2"
 			(at 37.846 48.26 0)
 			(effects
@@
 		)
 		(pin "2"
+			(alternate "Negative")
 		)
 		(pin "1"
+			(alternate "Positive")
 		)
 		(instances

Commit message: v0.1
Parts:
- added J5: Batt_Conn1, Battery:BatteryHolder_Keystone_1042_1x18650, symbol Connector_Generic:Conn_01x02
- added J6: Batt_Conn2, Battery:BatteryHolder_Keystone_1042_1x18650, symbol Connector_Generic:Conn_01x02
- added R12: 750R, LED_SMD:LED_1206_3216Metric_Pad1.42x1.75mm_HandSolder, symbol Device:R
- LED1: value GREEN -> RED; footprint SmartHomeFootprints:LED_1411 -> LED_SMD:LED_1206_3216Metric_Pad1.42x1.75mm_HandSolder; Store link https://hu.farnell.com/multicomp-pro/mp005918/led-green-225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 -> https://hu.farnell.com/kingbright/kptd-3216lvsurck/chip-led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
- R11: value 20R -> 10R; footprint Resistor_SMD:R_1210_3225Metric_Pad1.30x2.65mm_HandSolder -> LED_SMD:LED_1206_3216Metric_Pad1.42x1.75mm_HandSolder; Store link https://hu.farnell.com/vishay/crcw121020r0fkea/res-20r-1-0-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 -> https://hu.farnell.com/panasonic/erj8geyj100v/res-10r-5-0-2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
Connections:
- net GND: now also J6.1 (Pin_1)
- net at R11.2: now also R12.1; no longer LED1.2 (A)
- net at C13.1, J3.2 (Pin_2), U3.1 (IN): now also J5.2 (Pin_2)
- new net: J5.1 (Pin_1), J6.2 (Pin_2)
- new net: LED1.2 (A), R12.2
Other:
- note added: "MCU tápellátás"
- note removed: "MC tápellátás"
- moved on the sheet: C13, C14, J3, J4, LED1, R10, R11, U3

Commit message: v0.1
Parts:
- added J10, J7: Batt_Conn1, Battery:BatteryHolder_Keystone_1042_1x18650, symbol Connector_Generic:Conn_01x02
- added J11, J12, J8, J9: Batt_Conn2, Battery:BatteryHolder_Keystone_1042_1x18650, symbol Connector_Generic:Conn_01x02
Connections:
- net GND: now also J10.1 (Pin_1), J11.1 (Pin_1), J12.1 (Pin_1), J7.1 (Pin_1), J8.1 (Pin_1), J9.1 (Pin_1)
- new net: J7.2 (Pin_2), J8.2 (Pin_2), J9.2 (Pin_2)
- new net: J10.2 (Pin_2), J11.2 (Pin_2), J12.2 (Pin_2)
Other:
- note added: "MCU tápellátás (Batt measure missing)"
- note removed: "MCU tápellátás"

Commit message: v0.1
Parts:
- added U4: PAM2421AECADJR, symbol SmartHomeSymbols:PAM2421AECADJR
Connections:
- net at J7.2 (Pin_2), J8.2 (Pin_2), J9.2 (Pin_2): now also U4.5 (VIN)
Changed lines of the file:
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@@
+	)
+	(junction
+		(at 95.25 81.28)
+		(diameter 0)
+		(color 0 0 0 0)
 	)
 	(junction
@@
 		(pts
 			(xy 198.12 97.79) (xy 218.44 97.79)
+		)
+		(stroke
+			(width 0)
+			(type default)
+		)
+	)
+	(wire
+		(pts
+			(xy 119.38 81.28) (xy 95.25 81.28)
 		)
 		(stroke
@@
 					(unit 1)
 				)
+			)
+		)
+	)
+	(symbol
+		(lib_id "SmartHomeSymbols:PAM2421AECADJR")
+		(at 109.22 83.82 0)
+		(unit 1)
+		(exclude_from_sim no)
+		(in_bom yes)
+		(on_board yes)
+		(dnp no)
+		(property "Reference" "U4"
+			(at 132.08 98.044 0)
+			(effects
+				(font
+					(size 1.27 1.27)
+				)
+			)
+		)
+		(property "Value" "PAM2421AECADJR"
+			(at 132.08 100.584 0)
+			(effects
+				(font
+					(size 1.27 1.27)
+				)
+			)
+		)
+		(property "Footprint" ""
+			(at 109.22 83.82 0)
+			(effects
+				(font
+					(size 1.27 1.27)
+				)
+				(hide yes)
+			)
+		)
+		(property "Datasheet" ""
+			(at 109.22 83.82 0)
+			(effects
+				(font
+					(size 1.27 1.27)
+				)
+				(hide yes)
+			)
+		)
+		(property "Description" ""
+			(at 109.22 83.82 0)
+			(effects
+				(font
+					(size 1.27 1.27)
+				)
+				(hide yes)
+			)
+		)
+		(pin "2"
+		)
+		(pin "4"
+		)
+		(pin "3"
+		)
+		(pin "1"
+		)
+		(pin "5"
+		)
+		(instances
+			(project "WindowOpener"
+				(path "/9cc66d3b-a4f0-4570-ad5d-091fde92d938/9855627f-fa2d-4bc2-9342-1b3aeb423b2c"
+					(reference "U4")
+					(unit 1)
+				)

Commit message: v0.2
Parts:
- removed J10: Batt_Conn1, Battery:BatteryHolder_Keystone_1042_1x18650, symbol Connector_Generic:Conn_01x02
- added C15, C17: 2u2F, Capacitor_SMD:C_1206_3216Metric_Pad1.33x1.80mm_HandSolder, symbol Device:C
- added C16, C18: 10uF, Capacitor_SMD:C_1206_3216Metric_Pad1.33x1.80mm_HandSolder, symbol Device:C
- added D1, D2: 1A40V, SmartHomeFootprints:1N5819HW-7-F, symbol Device:D_Schottky
- added J10: Motor1, Connector_PinHeader_2.54mm:PinHeader_1x02_P2.54mm_Vertical, symbol Connector:Conn_01x02_Pin
- added J13: Batt_Conn, Battery:BatteryHolder_Keystone_1042_1x18650, symbol Connector_Generic:Conn_01x02
- added J14: Motor2, Connector_PinHeader_2.54mm:PinHeader_1x02_P2.54mm_Vertical, symbol Connector:Conn_01x02_Pin
- added L1, L2: 10uH, Inductor_SMD:L_1210_3225Metric_Pad1.42x2.65mm_HandSolder, symbol Device:L
- added R13, R17: 4k3, Resistor_SMD:R_1206_3216Metric_Pad1.30x1.75mm_HandSolder, symbol Device:R
- added R14, R18: 82k, Resistor_SMD:R_1206_3216Metric_Pad1.30x1.75mm_HandSolder, symbol Device:R
- added R15, R19: 470R, Resistor_SMD:R_1206_3216Metric_Pad1.30x1.75mm_HandSolder, symbol Device:R
- added R16, R20: 10k, Resistor_SMD:R_2010_5025Metric_Pad1.40x2.65mm_HandSolder, symbol Device:R
- added U5, U6: DRV8220DRL, Package_TO_SOT_SMD:SOT-563, symbol Driver_Motor:DRV8220DRL
- added U7: MIC2288YD5-TR, Package_TO_SOT_SMD:TSOT-23-5_HandSoldering, symbol SmartHomeSymbols:PAM2421AECADJR
- C13: footprint Capacitor_SMD:C_2220_5750Metric_Pad1.97x5.40mm_HandSolder -> Capacitor_SMD:C_1206_3216Metric_Pad1.33x1.80mm_HandSolder; Store link https://hu.farnell.com/chemi-con/kts500b106m55n0t00/cap-mlc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 -> https://hu.farnell.com/multicomp-pro/1206x106k160ct/cap-10-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
- J11, J12, J4, J6, J8, J9: value Batt_Conn2 -> Batt_Conn
- J3, J5, J7: value Batt_Conn1 -> Batt_Conn
- R11, R12: footprint LED_SMD:LED_1206_3216Metric_Pad1.42x1.75mm_HandSolder -> Resistor_SMD:R_1206_3216Metric_Pad1.30x1.75mm_HandSolder
- U4: value PAM2421AECADJR -> MIC2288YD5-TR; footprint (none) -> Package_TO_SOT_SMD:TSOT-23-5_HandSoldering; Store link (none) -> https://hu.farnell.com/microchip/mic2288yd5-tr/switching-re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
Connections:
- net GND: now also J11.2 (Pin_1), J12.2 (Pin_1), J4.2 (Pin_1), J6.2 (Pin_1), J7.2 (Pin_1), J8.2 (Pin_1), J9.2 (Pin_1), U4.2 (GND), C15.2, C16.2, C17.2, C18.2, J13.2 (Pin_1), R16.2, R20.2, U5.3 (GND), U6.3 (GND), U7.2 (GND); no longer J11.1 (Pin_1), J12.1 (Pin_1), J4.1 (Pin_1), J6.1 (Pin_1), J7.1 (Pin_1), J8.1 (Pin_1), J9.1 (Pin_1)
- net at J3.1 (Pin_2): now also C13.1, J5.1 (Pin_2), U3.1 (IN); no longer J4.2 (Pin_2)
- net at U4.1 (SW): now also D1.2 (A), L1.2
- net at U4.3 (FB): now also R15.2, R16.1
- net at U4.4 (EN): now also J7.1 (Pin_2), J8.1 (Pin_2), J9.1 (Pin_2), U4.5 (VIN), C15.1, L1.1
- new net: D2.2 (A), L2.2, U7.1 (SW)
- new net: J5.2 (Pin_1), J6.1 (Pin_2)
- new net: R13.2, R14.1
- new net: R17.2, R18.1
- new net: C17.1, J11.1 (Pin_2), J12.1 (Pin_2), J13.1 (Pin_2), L2.1, U7.4 (EN), U7.5 (VIN)
- new net: J10.1 (Pin_2), U5.6 (OUT1)
- new net: J10.2 (Pin_1), U5.4 (OUT2)
- new net: J14.1 (Pin_2), U6.6 (OUT1)
- new net: J14.2 (Pin_1), U6.4 (OUT2)
- new net: R18.2, R19.1
- new net: R19.2, R20.1, U7.3 (FB)
- new net: J3.2 (Pin_1), J4.1 (Pin_2)
- new net: R14.2, R15.1
- new net 12VM1: C16.1, D1.1 (K), R13.1, U5.5 (VM)
- new net 12VM2: C18.1, D2.1 (K), R17.1, U6.5 (VM)
- new net IN1_1: U5.1 (IN1)
- new net IN1_2: U6.1 (IN1)
- new net IN2_1: U5.2 (IN2)
- new net IN2_2: U6.2 (IN2)
Other:
- note added: "Motor1 Power+Driver"
- note added: "Motor2 Power+Driver"
- moved on the sheet: C13, C14, J3, LED1, R10, R11, R12, U3, U4

Commit message: v0.3
Connections:
- net ADC1: now reaches C13.1, J3.1 (Pin_2), J5.1 (Pin_2), U3.1 (IN)
- net ADC4: now reaches J5.2 (Pin_1), J6.1 (Pin_2)
- net ADC6: now reaches C17.1, J11.1 (Pin_2), J12.1 (Pin_2), J13.1 (Pin_2), L2.1, U7.4 (EN), U7.5 (VIN)
- net ADC2: now reaches J3.2 (Pin_1), J4.1 (Pin_2)
- net ADC5: now reaches C15.1, J7.1 (Pin_2), J8.1 (Pin_2), J9.1 (Pin_2), L1.1, U4.4 (EN), U4.5 (VIN)
Other:
- moved on the sheet: J4, J6
