File: WindowOpener/power.kicad_sch (KiCad schematic)
At the start: 39 parts, among them J10 Motor1, J11 Batt_Conn, J12 Batt_Conn, J13 Batt_Conn, J14 Motor2, J3 Batt_Conn, J4 Batt_Conn, J5 Batt_Conn, J6 Batt_Conn, J7 Batt_Conn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

Commit message: v0.5
Parts:
- added R41, R42, R43, R44, R45, R46, R47: 1k, Resistor_SMD:R_2010_5025Metric_Pad1.40x2.65mm_HandSolder, symbol Device:R
- U5, U6: Store link (none) -> https://www.ti.com/product/DRV8220?login-check=true#order-q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
Connections:
- net ADC1: now also R41.1, R42.2; no longer C13.1, J3.1 (Pin_2), J5.1 (Pin_2), U3.1 (IN)
- net ADC2: now also R44.1, R45.2; no longer C15.1, J7.1 (Pin_2), J8.1 (Pin_2), J9.1 (Pin_2), L1.1, U4.4 (EN), U4.5 (VIN)
- net ADC3: now also R46.1, R47.2; no longer C17.1, J11.1 (Pin_2), J12.1 (Pin_2), J13.1 (Pin_2), L2.1, U7.4 (EN), U7.5 (VIN)
- net GND: now also R42.1, R45.1, R47.1
- new net: C13.1, J3.1 (Pin_2), J5.1 (Pin_2), R43.2, U3.1 (IN)
- new net: C17.1, J11.1 (Pin_2), J12.1 (Pin_2), J13.1 (Pin_2), L2.1, R46.2, U7.4 (EN), U7.5 (VIN)
- new net: R41.2, R43.1
- new net: C15.1, J7.1 (Pin_2), J8.1 (Pin_2), J9.1 (Pin_2), L1.1, R44.2, U4.4 (EN), U4.5 (VIN)
Other:
- moved on the sheet: C17, C18, D2, J11, J12, J13, J14, J7, J8, J9, L2, R17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

Commit message: v0.6
Parts:
- added R51, R52, R53, R56: 330R, Resistor_SMD:R_2010_5025Metric_Pad1.40x2.65mm_HandSolder, symbol Device:R
- added R54, R55, R57, R58: 100R, Resistor_SMD:R_2010_5025Metric_Pad1.40x2.65mm_HandSolder, symbol Device:R
- U5, U6: Store link https://www.ti.com/product/DRV8220?login-check=true#order-q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 -> https://hu.mouser.com/ProductDetail/Texas-Instruments/DRV82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
Connections:
- net GND: now also R54.1, R55.1, R57.1, R58.1
- net at J10.1 (Pin_2), U5.6 (OUT1): now also R52.2
- net at J10.2 (Pin_1), U5.4 (OUT2): now also R51.2
- net at J14.1 (Pin_2), U6.6 (OUT1): now also R56.2
- net at J14.2 (Pin_1), U6.4 (OUT2): now also R53.2
- new net ADC4: R51.1, R54.2
- new net ADC5: R52.1, R58.2
- new net ADC6: R53.1, R55.2
- new net ADC7: R56.1, R57.2
Other:
- moved on the sheet: C17, C18, D2, J10, J11, J12, J13, J14, L2, R17, R18, R19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

Commit message: v0.7
Parts:
- removed J13, J9: Batt_Conn, Battery:BatteryHolder_Keystone_1042_1x18650, symbol Connector_Generic:Conn_01x02
Other:
- moved on the sheet: J11, J12, J7, J8, R44, R45, R46, R47

Commit message: v1.0
Parts:
- renumbered R47 to R44, R46 to R45, R44 to R46, R45 to R47
Changed lines of the file:
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@@
 		(on_board yes)
 		(dnp no)
-		(property "Reference" "R47"
+		(property "Reference" "R44"
 			(at 170.18 41.91 90)
 			(effects
@@
 			(project "WindowOpener"
 				(path "/9cc66d3b-a4f0-4570-ad5d-091fde92d938/9855627f-fa2d-4bc2-9342-1b3aeb423b2c"
-					(reference "R47")
+					(reference "R44")
 					(unit 1)
 				)
@@
 		(on_board yes)
 		(dnp no)
-		(property "Reference" "R44"
+		(property "Reference" "R46"
 			(at 35.56 87.63 90)
 			(effects
@@
 			(project "WindowOpener"
 				(path "/9cc66d3b-a4f0-4570-ad5d-091fde92d938/9855627f-fa2d-4bc2-9342-1b3aeb423b2c"
-					(reference "R44")
+					(reference "R46")
 					(unit 1)
 				)
@@
 		(on_board yes)
 		(dnp no)
-		(property "Reference" "R46"
+		(property "Reference" "R45"
 			(at 170.18 31.75 90)
 			(effects
@@
 			(project "WindowOpener"
 				(path "/9cc66d3b-a4f0-4570-ad5d-091fde92d938/9855627f-fa2d-4bc2-9342-1b3aeb423b2c"
-					(reference "R46")
+					(reference "R45")
 					(unit 1)
 				)
@@
 		(on_board yes)
 		(dnp no)
-		(property "Reference" "R45"
+		(property "Reference" "R47"
 			(at 35.56 97.79 90)
 			(effects
@@
 			(project "WindowOpener"
 				(path "/9cc66d3b-a4f0-4570-ad5d-091fde92d938/9855627f-fa2d-4bc2-9342-1b3aeb423b2c"
-					(reference "R45")
+					(reference "R47")
 					(unit 1)
 				)

Commit message: v1.0.1
Parts:
- R11: Store link https://hu.farnell.com/panasonic/erj8geyj100v/res-10r-5-0-2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 -> https://hu.farnell.com/multicomp-pro/mcwr12x10r0ftl/res-10r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
Changed lines of the file:
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@@
 			)
 		)
-		(property "Datasheet" "https://4donline.ihs.com/images/VipMasterIC/IC/PANA/PANA-S-A0017042869/PANA-S-A0017226461-1.pdf?hkey=6D3A4C79FDBF58556ACFDE234799DDF0"
+		(property "Datasheet" "https://www.farnell.com/datasheets/3680671.pdf"
 			(at 120.65 35.56 0)
 			(effects
@@
 			)
 		)
-		(property "Store link" "https://hu.farnell.com/panasonic/erj8geyj100v/res-10r-5-0-25w-1206-thick-film/dp/4147891"
+		(property "Store link" "https://hu.farnell.com/multicomp-pro/mcwr12x10r0ftl/res-10r-1-0-25w-1206-thick-film/dp/2447457"
 			(at 120.65 35.56 90)
 			(effects
