File: WindowOpener/sensors.kicad_sch (KiCad schematic)
At the start: 3 parts, among them U2 AM2302, U8 TSOP348xx

Commit message: v0.4
Parts:
- R5: value 100R -> 1k
Changed lines of the file:
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@@
 			)
 		)
-		(property "Value" "100R"
+		(property "Value" "1k"
 			(at 54.61 38.1 90)
 			(effects

Commit message: v0.5
Parts:
- U8: Store link (none) -> https://hu.farnell.com/vishay/tsop34838/ir-receiver-45m-0-0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
Changed lines of the file:
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@@
+			)
+		)
+		(property "Store link" "https://hu.farnell.com/vishay/tsop34838/ir-receiver-45m-0-08mw-m2-side/dp/4913139"
+			(at 46.99 82.55 0)
+			(effects
+				(font
+					(size 1.27 1.27)
+				)
+				(hide yes)
 			)
 		)
