File: WindowOpener/leds.kicad_sch (KiCad schematic)
At the start: 24 parts

Commit message: v0.6
Parts:
- added LED8: RED, LED_SMD:LED_1206_3216Metric_Pad1.42x1.75mm_HandSolder, symbol Device:LED
- added R48: 750R, Resistor_SMD:R_1206_3216Metric_Pad1.30x1.75mm_HandSolder, symbol Device:R
- added R49: 10R, Resistor_SMD:R_1206_3216Metric_Pad1.30x1.75mm_HandSolder, symbol Device:R
- added R50: 15R, Resistor_SMD:R_1210_3225Metric_Pad1.30x2.65mm_HandSolder, symbol Device:R
Connections:
- net GND: now also LED8.1 (K)
- new net: LED8.2 (A), R50.1
- new net: R48.1, R49.2
- new net: R49.1, R50.2
- new net LED8: R48.2

Commit message: v1.0.1
Parts:
- R24, R27, R30, R33, R36, R39, R49: Store link https://hu.farnell.com/panasonic/erj8geyj100v/res-10r-5-0-2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 -> https://hu.farnell.com/multicomp-pro/mcwr12x10r0ftl/res-10r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
Changed lines of the file:
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@@
 			)
 		)
-		(property "Datasheet" "https://4donline.ihs.com/images/VipMasterIC/IC/PANA/PANA-S-A0017042869/PANA-S-A0017226461-1.pdf?hkey=6D3A4C79FDBF58556ACFDE234799DDF0"
+		(property "Datasheet" "https://www.farnell.com/datasheets/3680671.pdf"
 			(at 100.33 46.99 0)
 			(effects
@@
 			)
 		)
-		(property "Store link" "https://hu.farnell.com/panasonic/erj8geyj100v/res-10r-5-0-25w-1206-thick-film/dp/4147891"
+		(property "Store link" "https://hu.farnell.com/multicomp-pro/mcwr12x10r0ftl/res-10r-1-0-25w-1206-thick-film/dp/2447457"
 			(at 100.33 46.99 90)
 			(effects
@@
 			)
 		)
-		(property "Datasheet" "https://4donline.ihs.com/images/VipMasterIC/IC/PANA/PANA-S-A0017042869/PANA-S-A0017226461-1.pdf?hkey=6D3A4C79FDBF58556ACFDE234799DDF0"
+		(property "Datasheet" "https://www.farnell.com/datasheets/3680671.pdf"
 			(at 116.84 46.99 0)
 			(effects
@@
 			)
 		)
-		(property "Store link" "https://hu.farnell.com/panasonic/erj8geyj100v/res-10r-5-0-25w-1206-thick-film/dp/4147891"
+		(property "Store link" "https://hu.farnell.com/multicomp-pro/mcwr12x10r0ftl/res-10r-1-0-25w-1206-thick-film/dp/2447457"
 			(at 116.84 46.99 90)
 			(effects
@@
 			)
 		)
-		(property "Datasheet" "https://4donline.ihs.com/images/VipMasterIC/IC/PANA/PANA-S-A0017042869/PANA-S-A0017226461-1.pdf?hkey=6D3A4C79FDBF58556ACFDE234799DDF0"
+		(property "Datasheet" "https://www.farnell.com/datasheets/3680671.pdf"
 			(at 83.82 46.99 0)
 			(effects
@@
 			)
 		)
-		(property "Store link" "https://hu.farnell.com/panasonic/erj8geyj100v/res-10r-5-0-25w-1206-thick-film/dp/4147891"
+		(property "Store link" "https://hu.farnell.com/multicomp-pro/mcwr12x10r0ftl/res-10r-1-0-25w-1206-thick-film/dp/2447457"
 			(at 83.82 46.99 90)
 			(effects
@@
 			)
 		)
-		(property "Datasheet" "https://4donline.ihs.com/images/VipMasterIC/IC/PANA/PANA-S-A0017042869/PANA-S-A0017226461-1.pdf?hkey=6D3A4C79FDBF58556ACFDE234799DDF0"
+		(property "Datasheet" "https://www.farnell.com/datasheets/3680671.pdf"
 			(at 36.83 46.99 0)
 			(effects
@@
 			)
 		)
-		(property "Store link" "https://hu.farnell.com/panasonic/erj8geyj100v/res-10r-5-0-25w-1206-thick-film/dp/4147891"
+		(property "Store link" "https://hu.farnell.com/multicomp-pro/mcwr12x10r0ftl/res-10r-1-0-25w-1206-thick-film/dp/2447457"
 			(at 36.83 46.99 90)
 			(effects
@@
 			)
 		)
-		(property "Datasheet" "https://4donline.ihs.com/images/VipMasterIC/IC/PANA/PANA-S-A0017042869/PANA-S-A0017226461-1.pdf?hkey=6D3A4C79FDBF58556ACFDE234799DDF0"
+		(property "Datasheet" "https://www.farnell.com/datasheets/3680671.pdf"
 			(at 67.31 46.99 0)
 			(effects
@@
 			)
 		)
-		(property "Store link" "https://hu.farnell.com/panasonic/erj8geyj100v/res-10r-5-0-25w-1206-thick-film/dp/4147891"
+		(property "Store link" "https://hu.farnell.com/multicomp-pro/mcwr12x10r0ftl/res-10r-1-0-25w-1206-thick-film/dp/2447457"
 			(at 67.31 46.99 90)
 			(effects
@@
 			)
 		)
-		(property "Datasheet" "https://4donline.ihs.com/images/VipMasterIC/IC/PANA/PANA-S-A0017042869/PANA-S-A0017226461-1.pdf?hkey=6D3A4C79FDBF58556ACFDE234799DDF0"
+		(property "Datasheet" "https://www.farnell.com/datasheets/3680671.pdf"
 			(at 134.62 46.99 0)
 			(effects
@@
 			)
 		)
-		(property "Store link" "https://hu.farnell.com/panasonic/erj8geyj100v/res-10r-5-0-25w-1206-thick-film/dp/4147891"
+		(property "Store link" "https://hu.farnell.com/multicomp-pro/mcwr12x10r0ftl/res-10r-1-0-25w-1206-thick-film/dp/2447457"
 			(at 134.62 46.99 90)
 			(effects
@@
 			)
 		)
-		(property "Datasheet" "https://4donline.ihs.com/images/VipMasterIC/IC/PANA/PANA-S-A0017042869/PANA-S-A0017226461-1.pdf?hkey=6D3A4C79FDBF58556ACFDE234799DDF0"
+		(property "Datasheet" "https://www.farnell.com/datasheets/3680671.pdf"
 			(at 52.07 46.99 0)
 			(effects
@@
 			)
 		)
-		(property "Store link" "https://hu.farnell.com/panasonic/erj8geyj100v/res-10r-5-0-25w-1206-thick-film/dp/4147891"
+		(property "Store link" "https://hu.farnell.com/multicomp-pro/mcwr12x10r0ftl/res-10r-1-0-25w-1206-thick-film/dp/2447457"
 			(at 52.07 46.99 90)
 			(effects
