File: WindowOpener/WindowOpener.kicad_pcb (KiCad board)
At the start: 2 copper layers, 145 x 85 mm, 59 parts, among them J1 Conn_ST_STDC14, J2 UEXT_Host, J3 USB_C_Receptacle_USB2.0_16P, SW1 SW_Push, SW2 SW_SPDT_XKB, SW3 SW_SPDT_XKB, U1 STM32L152RCTxA, U2 AM2302, U6 MCP73831-2-OT, U7 NID5100GW, U8 NID5100GW, U9 LM1117DT-3.3, Y1 8MHz, Y2 32.768kHz

Commit message: v0.5
Parts:
- removed BATT1: Battery conn, Battery:BatteryHolder_Keystone_1042_1x18650
- removed C19: 0,1uF, Capacitor_SMD:C_1206_3216Metric_Pad1.33x1.80mm_HandSolder
- removed C20, C21: 1uF, Capacitor_SMD:C_2220_5750Metric_Pad1.97x5.40mm_HandSolder
- removed C22, C23: 0,47uF, Capacitor_SMD:C_2220_5750Metric_Pad1.97x5.40mm_HandSolder
- removed C24: 10uF, Capacitor_SMD:C_2220_5750Metric_Pad1.97x5.40mm_HandSolder
- removed G***: LOGO, LOGO
- removed SW3: SW_SPDT_XKB, Button_Switch_THT:SW_XKB_DM1-16UP-1
- removed U9: LM1117DT-3.3, Package_TO_SOT_SMD:TO-252-3_TabPin2
- added C13: 10uF, Capacitor_SMD:C_1206_3216Metric_Pad1.33x1.80mm_HandSolder, F.Cu at (-63.5, 43.5)
- added C14: 22uF, Capacitor_SMD:C_1206_3216Metric_Pad1.33x1.80mm_HandSolder, F.Cu at (-68.0, 43.5)
- added C15: 2u2F, Capacitor_SMD:C_1206_3216Metric_Pad1.33x1.80mm_HandSolder, F.Cu at (-42.4, 22.6)
- added C16: 10uF, Capacitor_SMD:C_1206_3216Metric_Pad1.33x1.80mm_HandSolder, F.Cu at (-42.4, 26.0)
- added C17: 2u2F, Capacitor_SMD:C_1206_3216Metric_Pad1.33x1.80mm_HandSolder, F.Cu at (-42.4, 29.3)
- added C18: 10uF, Capacitor_SMD:C_1206_3216Metric_Pad1.33x1.80mm_HandSolder, F.Cu at (-42.4, 32.7)
- added J10: Motor1, Connector_PinHeader_2.54mm:PinHeader_1x02_P2.54mm_Vertical, F.Cu at (-43.1, 45.0)
- added J11: Batt_Conn, Battery:BatteryHolder_Keystone_1042_1x18650, F.Cu at (264.0, 61.0)
- added J12: Batt_Conn, Battery:BatteryHolder_Keystone_1042_1x18650, F.Cu at (239.0, 61.0)
- added J13: Batt_Conn, Battery:BatteryHolder_Keystone_1042_1x18650, F.Cu at (214.3, 61.0)
- added J14: Motor2, Connector_PinHeader_2.54mm:PinHeader_1x02_P2.54mm_Vertical, F.Cu at (-38.5, 45.0)
- added J4: Batt_Conn, Battery:BatteryHolder_Keystone_1042_1x18650, F.Cu at (135.0, 61.0)
- added J5: Batt_Conn, Battery:BatteryHolder_Keystone_1042_1x18650, F.Cu at (159.0, 61.0)
- added J6: Batt_Conn, Battery:BatteryHolder_Keystone_1042_1x18650, F.Cu at (184.0, 61.0)
- added J7: Batt_Conn, Battery:BatteryHolder_Keystone_1042_1x18650, F.Cu at (82.0, 61.0)
- added J8: Batt_Conn, Battery:BatteryHolder_Keystone_1042_1x18650, F.Cu at (57.3, 61.0)
- added J9: Batt_Conn, Battery:BatteryHolder_Keystone_1042_1x18650, F.Cu at (33.0, 61.0)
- added L1: 10uH, Inductor_SMD:L_1210_3225Metric_Pad1.42x2.65mm_HandSolder, F.Cu at (-42.5, 51.9)
- added L2: 10uH, Inductor_SMD:L_1210_3225Metric_Pad1.42x2.65mm_HandSolder, F.Cu at (-42.5, 56.1)
- added LED1: RED, LED_SMD:LED_1206_3216Metric_Pad1.42x1.75mm_HandSolder, F.Cu at (-48.0, 90.0)
- added LED2: RED, LED_SMD:LED_1206_3216Metric_Pad1.42x1.75mm_HandSolder, F.Cu at (-24.6, -13.5)
- added LED3: RED, LED_SMD:LED_1206_3216Metric_Pad1.42x1.75mm_HandSolder, F.Cu at (-24.6, -10.1)
- added LED4: RED, LED_SMD:LED_1206_3216Metric_Pad1.42x1.75mm_HandSolder, F.Cu at (-24.6, -6.74)
- added LED5: RED, LED_SMD:LED_1206_3216Metric_Pad1.42x1.75mm_HandSolder, F.Cu at (-24.6, -3.35)
- added LED6: RED, LED_SMD:LED_1206_3216Metric_Pad1.42x1.75mm_HandSolder, F.Cu at (-24.6, 0.04)
- added LED7: RED, LED_SMD:LED_1206_3216Metric_Pad1.42x1.75mm_HandSolder, F.Cu at (-24.6, 3.44)
- added R23: 15R, Resistor_SMD:R_1210_3225Metric_Pad1.30x2.65mm_HandSolder, F.Cu at (-30.6, -13.1)
- added R24: 10R, Resistor_SMD:R_1206_3216Metric_Pad1.30x1.75mm_HandSolder, F.Cu at (-18.7, -13.6)
- added R25: 750R, Resistor_SMD:R_1206_3216Metric_Pad1.30x1.75mm_HandSolder, F.Cu at (-18.7, -10.2)
- added R26: 750R, Resistor_SMD:R_1206_3216Metric_Pad1.30x1.75mm_HandSolder, F.Cu at (-18.7, -6.93)
- added R27: 10R, Resistor_SMD:R_1206_3216Metric_Pad1.30x1.75mm_HandSolder, F.Cu at (-18.7, -3.62)
- added R28: 15R, Resistor_SMD:R_1210_3225Metric_Pad1.30x2.65mm_HandSolder, F.Cu at (-30.6, -8.89)
- added R29: 750R, Resistor_SMD:R_1206_3216Metric_Pad1.30x1.75mm_HandSolder, F.Cu at (-12.7, -13.6)
- added R30: 10R, Resistor_SMD:R_1206_3216Metric_Pad1.30x1.75mm_HandSolder, F.Cu at (-12.7, -10.2)
- added R31: 15R, Resistor_SMD:R_1210_3225Metric_Pad1.30x2.65mm_HandSolder, F.Cu at (-30.6, -4.68)
- added R32: 750R, Resistor_SMD:R_1206_3216Metric_Pad1.30x1.75mm_HandSolder, F.Cu at (-12.7, -6.93)
- added R33: 10R, Resistor_SMD:R_1206_3216Metric_Pad1.30x1.75mm_HandSolder, F.Cu at (-12.7, -3.62)
- added R34: 15R, Resistor_SMD:R_1210_3225Metric_Pad1.30x2.65mm_HandSolder, F.Cu at (-30.6, -0.47)
- added R35: 750R, Resistor_SMD:R_1206_3216Metric_Pad1.30x1.75mm_HandSolder, F.Cu at (-6.76, -13.6)
- added R36: 10R, Resistor_SMD:R_1206_3216Metric_Pad1.30x1.75mm_HandSolder, F.Cu at (-6.76, -10.2)
- added R37: 15R, Resistor_SMD:R_1210_3225Metric_Pad1.30x2.65mm_HandSolder, F.Cu at (-30.6, 3.73)
- added R38: 750R, Resistor_SMD:R_1206_3216Metric_Pad1.30x1.75mm_HandSolder, F.Cu at (-6.76, -6.93)
- added R39: 10R, Resistor_SMD:R_1206_3216Metric_Pad1.30x1.75mm_HandSolder, F.Cu at (-6.76, -3.62)
- added R40: 15R, Resistor_SMD:R_1210_3225Metric_Pad1.30x2.65mm_HandSolder, F.Cu at (-30.6, 7.95)
- added R41: 1k, Resistor_SMD:R_2010_5025Metric_Pad1.40x2.65mm_HandSolder, F.Cu at (-41.6, -13.1)
- added R42: 1k, Resistor_SMD:R_2010_5025Metric_Pad1.40x2.65mm_HandSolder, F.Cu at (-41.6, -8.89)
- added R43: 1k, Resistor_SMD:R_2010_5025Metric_Pad1.40x2.65mm_HandSolder, F.Cu at (-41.6, -4.68)
- added R44: 1k, Resistor_SMD:R_2010_5025Metric_Pad1.40x2.65mm_HandSolder, F.Cu at (-41.6, -0.47)
- added R45: 1k, Resistor_SMD:R_2010_5025Metric_Pad1.40x2.65mm_HandSolder, F.Cu at (-41.6, 3.73)
- added R46: 1k, Resistor_SMD:R_2010_5025Metric_Pad1.40x2.65mm_HandSolder, F.Cu at (-41.6, 7.95)
- added R47: 1k, Resistor_SMD:R_2010_5025Metric_Pad1.40x2.65mm_HandSolder, F.Cu at (-41.6, 12.2)
- added U3: AZ1117CH2-3.3, Package_TO_SOT_SMD:SOT-223-3_TabPin2, F.Cu at (-66.0, 50.9)
- added U4: MIC2288YD5-TR, Package_TO_SOT_SMD:TSOT-23-5_HandSoldering, F.Cu at (-41.9, 60.6)
- added U5: DRV8220DRL, Package_TO_SOT_SMD:SOT-563, F.Cu at (-37.7, 64.5)
- C6: footprint Capacitor_SMD:C_2220_5750Metric_Pad1.97x5.40mm_HandSolder -> Capacitor_SMD:C_1206_3216Metric_Pad1.33x1.80mm_HandSolder
- D1, D2: value LED -> 1A40V; footprint LED_SMD:LED_1206_3216Metric_Pad1.42x1.75mm_HandSolder -> SmartHomeFootprints:1N5819HW-7-F
- J3: value USB_C_Receptacle_USB2.0_16P -> Batt_Conn; footprint Connector_USB:USB_C_Receptacle_HRO_TYPE-C-31-M-12 -> Battery:BatteryHolder_Keystone_1042_1x18650
- R10: value 0R -> 15R; footprint Resistor_SMD:R_2010_5025Metric_Pad1.40x2.65mm_HandSolder -> Resistor_SMD:R_1210_3225Metric_Pad1.30x2.65mm_HandSolder
- R11: value 0R -> 10R; footprint Resistor_SMD:R_2010_5025Metric_Pad1.40x2.65mm_HandSolder -> Resistor_SMD:R_1206_3216Metric_Pad1.30x1.75mm_HandSolder
- R12: value 2k -> 750R; footprint Resistor_SMD:R_2010_5025Metric_Pad1.40x2.65mm_HandSolder -> Resistor_SMD:R_1206_3216Metric_Pad1.30x1.75mm_HandSolder
- R13: value 147R -> 4k3
- R14: value 50k -> 82k
- R15: value 50k -> 470R
- R16: value 50k -> 10k; footprint Resistor_SMD:R_1206_3216Metric_Pad1.30x1.75mm_HandSolder -> Resistor_SMD:R_2010_5025Metric_Pad1.40x2.65mm_HandSolder
- R17: value 50k -> 4k3
- R18: value 60R4 -> 82k
- R19: value 5k1 -> 470R; footprint Resistor_SMD:R_2010_5025Metric_Pad1.40x2.65mm_HandSolder -> Resistor_SMD:R_1206_3216Metric_Pad1.30x1.75mm_HandSolder
- R20: value 5k1 -> 10k
- R5: value 100R -> 1k
- U6: value MCP73831-2-OT -> DRV8220DRL; footprint Package_TO_SOT_SMD:SOT-23-5_HandSoldering -> Package_TO_SOT_SMD:SOT-563
- U7: value NID5100GW -> MIC2288YD5-TR; footprint Package_TO_SOT_SMD:SOT-363_SC-70-6_Handsoldering -> Package_TO_SOT_SMD:TSOT-23-5_HandSoldering
- U8: value NID5100GW -> TSOP348xx; footprint Package_TO_SOT_SMD:SOT-363_SC-70-6_Handsoldering -> OptoDevice:Vishay_MOLD-3Pin
- moved R12 273.1 mm to (-57.5, 88.0), turned to -90 degrees
- moved R11 264.2 mm to (-57.5, 83.0), turned to -90 degrees
- moved D1 259.4 mm to (-24.8, 29.2), turned to 0 degrees
- moved R10 258.2 mm to (-62.0, 83.0), turned to -90 degrees
- moved R13 255.0 mm to (-29.4, 22.9)
- moved R17 250.7 mm to (-29.4, 32.9)
- moved R15 246.8 mm to (-29.4, 29.6), turned to 0 degrees
- moved R20 243.0 mm to (-22.5, 21.0), turned to 0 degrees
- moved U6 242.9 mm to (-18.7, 35.5), turned to 0 degrees
- moved R18 240.7 mm to (-29.4, 36.2), turned to 0 degrees
- moved D2 237.6 mm to (-24.8, 32.3), turned to 0 degrees
- moved U8 233.5 mm to (-13.3, 16.7)
- moved R19 223.1 mm to (-29.4, 39.5)
- moved R14 222.2 mm to (-29.4, 26.2), turned to 0 degrees
- moved U7 222.1 mm to (-22.9, 25.4), turned to 0 degrees
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Connections:
- net /DHT22 renamed DHT22
- D1 pad 1: Net-(D1-K) -> 12VM1
- D2 pad 1: GND -> 12VM2
- R10 pad 1: Net-(U7-OUT) -> 3V3
- R10 pad 2: Net-(U9-VI) -> Net-(R10-Pad2)
- R11 pad 1: Net-(U8-OUT) -> Net-(R10-Pad2)
- R11 pad 2: Net-(U9-VI) -> Net-(R11-Pad2)
- R12 pad 1: GND -> Net-(R11-Pad2)
- R12 pad 2: Net-(U6-PROG) -> Net-(LED1-A)
- R13 pad 1: /Power+USB/VBUS -> 12VM1
- R13 pad 2: Net-(D1-A) -> Net-(R13-Pad2)
- R14 pad 1: GND -> Net-(R13-Pad2)
- R14 pad 2: Net-(U7-~{EN}) -> Net-(R14-Pad2)
- R15 pad 1: GND -> Net-(R14-Pad2)
- R15 pad 2: Net-(U8-~{EN}) -> Net-(U4-FB)
- R16 pad 1: Net-(U7-ST) -> Net-(U4-FB)
- R16 pad 2: Net-(U9-VI) -> GND
- R17 pad 1: Net-(U8-ST) -> 12VM2
- R17 pad 2: Net-(U9-VI) -> Net-(R17-Pad2)
- R18 pad 1: 3V3 -> Net-(R17-Pad2)
- R18 pad 2: Net-(D2-A) -> Net-(R18-Pad2)
- R19 pad 1: GND -> Net-(R18-Pad2)
- R19 pad 2: Net-(J3-CC2) -> Net-(U7-FB)
- R20 pad 1: GND -> Net-(U7-FB)
- R20 pad 2: Net-(J3-CC1) -> GND
- U1 pad 15: unconnected-(U1-PA1-Pad15) -> ADC1
- U1 pad 16: unconnected-(U1-PA2-Pad16) -> ADC2
- U1 pad 20: unconnected-(U1-PA4-Pad20) -> ADC3
- U1 pad 37: unconnected-(U1-PC6-Pad37) -> IN2_1
- U1 pad 38: unconnected-(U1-PC7-Pad38) -> LED3
- U1 pad 39: unconnected-(U1-PC8-Pad39) -> LED4
- U1 pad 40: unconnected-(U1-PC9-Pad40) -> LED5
- U1 pad 50: unconnected-(U1-PA15-Pad50) -> IN1_1
- U1 pad 51: unconnected-(U1-PC10-Pad51) -> LED6
- U1 pad 52: unconnected-(U1-PC11-Pad52) -> LED7
- U1 pad 61: unconnected-(U1-PB8-Pad61) -> IN1_2
- U1 pad 62: unconnected-(U1-PB9-Pad62) -> IN2_2
- U1 pad 9: unconnected-(U1-PC1-Pad9) -> LED2
- U6 pad 1: Net-(D1-K) -> IN1_2
- U6 pad 2: GND -> IN2_2
- U6 pad 3: Net-(SW3-A) -> GND
- U6 pad 4: /Power+USB/VBUS -> Net-(J14-Pin_1)
- U6 pad 5: Net-(U6-PROG) -> 12VM2
- U7 pad 1: /Power+USB/VBUS -> Net-(D2-A)
- U7 pad 3: Net-(U7-~{EN}) -> Net-(U7-FB)
- U7 pad 4: unconnected-(U7-Pad4) -> Net-(J11-Pin_2)
- U7 pad 5: Net-(U7-ST) -> Net-(J11-Pin_2)
- U8 pad 1: VBATT -> IR
- U8 pad 3: Net-(U8-~{EN}) -> 3V3
Routing:
- net 3V3: track 358.8 -> 15.5 mm, vias 8 -> 4
- net Net-(U9-VI): track 88.2 -> 0.00 mm
- net GND: track 161.4 -> 83.4 mm, vias 28 -> 15
- net Net-(BATT1-Pin_2): track 60.5 -> 0.00 mm, vias 2 -> 0
- net Net-(SW3-A): track 12.5 -> 0.00 mm, vias 2 -> 0
- net Net-(J3-CC1): track 12.2 -> 0.00 mm
- net Net-(D1-A): track 12.0 -> 0.00 mm
- net Net-(J3-CC2): track 10.9 -> 0.00 mm
- net Net-(U7-ST): track 10.6 -> 0.00 mm
- net Net-(D2-A): track 10.1 -> 0.00 mm, vias 2 -> 0
- net Net-(U8-ST): track 8.63 -> 0.00 mm
- net Net-(D1-K): track 8.31 -> 0.00 mm
- net Net-(U7-OUT): track 7.77 -> 0.00 mm
- net Net-(U6-PROG): track 7.69 -> 0.00 mm
- net VBATT: track 7.45 -> 0.00 mm
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- removed copper zone on F.Cu, net /Power+USB/VBUS
- removed copper zone on F.Cu, net 3V3
- removed copper zone on B.Cu, net GND
Other:
- board outline removed
- board text removed: "Battery"
- board text removed: "Charge"
- board text removed: "Charging"
- board text removed: "Power"
- board text removed: "Somogyi Tamás Szilágyi Péter"
- board text removed: "USB"

Commit message: v0.6
Parts:
- added LED8: RED, LED_SMD:LED_1206_3216Metric_Pad1.42x1.75mm_HandSolder, F.Cu at (265.5, 173.5)
- added R48: 750R, Resistor_SMD:R_1206_3216Metric_Pad1.30x1.75mm_HandSolder, F.Cu at (273.6, 168.0)
- added R49: 10R, Resistor_SMD:R_1206_3216Metric_Pad1.30x1.75mm_HandSolder, F.Cu at (273.6, 173.5)
- added R50: 15R, Resistor_SMD:R_1210_3225Metric_Pad1.30x2.65mm_HandSolder, F.Cu at (273.6, 179.5)
- added R51: 330R, Resistor_SMD:R_2010_5025Metric_Pad1.40x2.65mm_HandSolder, F.Cu at (69.6, 147.2)
- added R52: 330R, Resistor_SMD:R_2010_5025Metric_Pad1.40x2.65mm_HandSolder, F.Cu at (69.6, 153.7)
- added R53: 330R, Resistor_SMD:R_2010_5025Metric_Pad1.40x2.65mm_HandSolder, F.Cu at (263.7, 147.0)
- added R54: 100R, Resistor_SMD:R_2010_5025Metric_Pad1.40x2.65mm_HandSolder, F.Cu at (78.5, 147.2)
- added R55: 100R, Resistor_SMD:R_2010_5025Metric_Pad1.40x2.65mm_HandSolder, F.Cu at (263.7, 153.3)
- added R56: 330R, Resistor_SMD:R_2010_5025Metric_Pad1.40x2.65mm_HandSolder, F.Cu at (273.6, 147.0)
- added R57: 100R, Resistor_SMD:R_2010_5025Metric_Pad1.40x2.65mm_HandSolder, F.Cu at (273.6, 153.3)
- added R58: 100R, Resistor_SMD:R_2010_5025Metric_Pad1.40x2.65mm_HandSolder, F.Cu at (78.5, 153.7)
- moved R45 331.3 mm to (254.1, 153.3)
- moved R44 330.4 mm to (254.1, 147.0)
- moved LED7 329.4 mm to (257.5, 173.5)
- moved J14 328.0 mm to (280.0, 123.1)
- moved R40 328.0 mm to (248.9, 179.5), turned to 180 degrees
- moved C18 317.7 mm to (260.5, 128.5)
- moved L2 317.6 mm to (268.0, 123.0)
- moved C17 317.1 mm to (260.5, 123.0), turned to 180 degrees
- moved R39 311.1 mm to (248.9, 173.5)
- moved R38 309.8 mm to (248.9, 168.0)
- moved U7 309.0 mm to (268.0, 129.5)
- moved D2 308.6 mm to (266.0, 135.6)
- moved U6 305.0 mm to (268.0, 139.6)
- moved R20 301.0 mm to (254.0, 140.0)
- moved R29 299.2 mm to (257.2, 115.5)
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Connections:
- U1 pad 10: unconnected-(U1-PC2-Pad10) -> ADC4
- U1 pad 11: unconnected-(U1-PC3-Pad11) -> ADC5
- U1 pad 24: unconnected-(U1-PC4-Pad24) -> ADC6
- U1 pad 25: unconnected-(U1-PC5-Pad25) -> ADC7
- U1 pad 53: unconnected-(U1-PC12-Pad53) -> LED8
Routing:
- net /MISO: track 66.7 -> 0.00 mm, vias 2 -> 0
- net /CSEL: track 61.4 -> 0.00 mm, vias 2 -> 0
- net /MOSI: track 60.9 -> 0.00 mm, vias 2 -> 0
- net DHT22: track 50.9 -> 0.00 mm, vias 2 -> 0
- net /SCK: track 49.3 -> 0.00 mm, vias 2 -> 0
- net 3V3: track 15.5 -> 0.03 mm, vias 4 -> 0
- net GND: track 83.4 -> 70.9 mm, vias 15 -> 12
- net Net-(J2-SCL): track 8.98 -> 0.00 mm
- net Net-(J2-TXD): track 8.45 -> 0.00 mm
- net Net-(J2-SDA): track 7.17 -> 0.00 mm
Other:
- board outline added: 246 x 175 mm

Commit message: v0.7
Parts:
- removed J13, J9: Batt_Conn, Battery:BatteryHolder_Keystone_1042_1x18650
- Y2: footprint Crystal:Crystal_C26-LF_D2.1mm_L6.5mm_Horizontal -> Crystal:Crystal_C26-LF_D2.1mm_L6.5mm_Vertical
- moved J4 106.1 mm to (247.5, 102.8), turned to 0 degrees
- moved J12 99.1 mm to (334.5, 109.5), turned to -90 degrees
- moved LED4 96.0 mm to (331.6, 158.0)
- moved J3 93.1 mm to (247.1, 76.8), turned to 0 degrees
- moved R31 91.7 mm to (322.1, 158.0), turned to 180 degrees
- moved R30 77.7 mm to (314.1, 158.0), turned to 180 degrees
- moved J14 72.4 mm to (344.0, 157.0)
- moved R29 64.8 mm to (306.1, 158.0), turned to 180 degrees
- moved J7 63.6 mm to (61.2, 102.8), turned to 180 degrees
- moved R26 63.6 mm to (228.8, 123.8)
- moved R27 63.6 mm to (220.4, 123.8)
- moved R28 63.6 mm to (212.4, 123.8)
- moved J11 59.8 mm to (306.5, 109.6), turned to -90 degrees
- moved LED3 44.1 mm to (201.9, 123.8), turned to 0 degrees
- moved J6 42.3 mm to (153.5, 102.8), turned to 0 degrees
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Routing:
- net /SWCLK: track 87.4 -> 0.00 mm, vias 1 -> 0
- net /SWDIO: track 79.4 -> 0.00 mm, vias 1 -> 0
- net GND: track 70.9 -> 5.37 mm, vias 12 -> 3
- net /RESET: track 57.8 -> 0.28 mm
- net Net-(U1-BOOT0): track 50.1 -> 0.00 mm, vias 2 -> 0
- net GNDA: track 32.7 -> 0.00 mm, vias 2 -> 0
- net VDDA: track 29.1 -> 0.18 mm, vias 2 -> 0
- net /SOSC_IN: track 18.3 -> 0.00 mm, vias 2 -> 0
- net /OSC_IN: track 14.7 -> 0.00 mm
- net Net-(C9-Pad1): track 10.6 -> 0.00 mm
- net Net-(J1-~{RST}): track 10.6 -> 0.00 mm, vias 2 -> 0
- net Net-(SW2-A): track 8.55 -> 0.00 mm
- net Net-(J1-VCP_RX): track 7.73 -> 0.00 mm
- net Net-(C11-Pad1): track 6.77 -> 0.00 mm
- net Net-(J1-JTDI/NC): track 5.65 -> 0.20 mm
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Other:
- board size 246 x 175 mm -> 335.5 x 108 mm

Commit message: v1.0
Parts:
- moved U8 80.7 mm to (196.6, 149.4)
- moved LED3 26.3 mm to (222.7, 107.7)
- moved R26 26.3 mm to (249.6, 107.7)
- moved R28 26.3 mm to (233.1, 107.7)
- moved R27 26.3 mm to (241.1, 107.7)
- moved C8 25.0 mm to (148.8, 144.7)
- moved C2 24.8 mm to (213.1, 121.9)
- moved D2 24.8 mm to (287.4, 122.5)
- moved C1 24.8 mm to (213.1, 128.3)
- moved C10 24.8 mm to (171.9, 120.2)
- moved C11 24.8 mm to (190.5, 112.4)
- moved C12 24.8 mm to (173.7, 114.0)
- moved C13 24.8 mm to (146.7, 128.6)
- moved C14 24.8 mm to (152.7, 128.6)
- moved C15 24.8 mm to (60.3, 120.5)
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Connections:
- R44 pad 1: ADC2 -> GND
- R44 pad 2: Net-(J7-Pin_2) -> ADC3
- R45 pad 1: GND -> ADC3
- R45 pad 2: ADC2 -> Net-(J11-Pin_2)
- R46 pad 1: ADC3 -> ADC2
- R46 pad 2: Net-(J11-Pin_2) -> Net-(J7-Pin_2)
- R47 pad 2: ADC3 -> ADC2
- U1 pad 28: unconnected-(U1-PB2-Pad28) -> IR
- U1 pad 38: LED3 -> LED5
- U1 pad 40: LED5 -> LED3
- U1 pad 42: unconnected-(U1-PA9-Pad42) -> LED7
- U1 pad 43: unconnected-(U1-PA10-Pad43) -> LED8
- U1 pad 51: LED6 -> unconnected-(U1-PC10-Pad51)
- U1 pad 52: LED7 -> unconnected-(U1-PC11-Pad52)
- U1 pad 53: LED8 -> LED6
Routing:
- net GND: track 5.37 -> 350.5 mm, vias 3 -> 36
- net IN2_1: track 0.00 -> 205.1 mm, vias 0 -> 2
- net Net-(J7-Pin_2): track 0.00 -> 185.3 mm
- net LED5: track 0.00 -> 184.8 mm, vias 0 -> 2
- net IN1_1: track 0.00 -> 164.3 mm, vias 0 -> 4
- net Net-(J3-Pin_2): track 0.00 -> 159.6 mm, vias 0 -> 2
- net Net-(J11-Pin_2): track 0.00 -> 150.0 mm, vias 0 -> 4
- net ADC6: track 0.00 -> 145.3 mm, vias 0 -> 6
- net LED4: track 0.00 -> 141.6 mm, vias 0 -> 2
- net ADC3: track 0.00 -> 139.5 mm, vias 0 -> 4
- net ADC7: track 0.00 -> 138.7 mm, vias 0 -> 6
- net ADC2: track 0.00 -> 124.6 mm, vias 0 -> 2
- net Net-(J14-Pin_2): track 0.00 -> 108.1 mm, vias 0 -> 1
- net ADC4: track 0.00 -> 107.6 mm, vias 0 -> 2
- net LED8: track 0.00 -> 107.4 mm, vias 0 -> 2
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- added copper zone on F.Cu, net 3V3
- added copper zone on B.Cu, net GND

Commit message: v1.0.2
Parts:
- added H1: MountingHole, MountingHole:MountingHole_5.3mm_M5, F.Cu at (42.0, 151.2)
- added H2: MountingHole, MountingHole:MountingHole_5.3mm_M5, F.Cu at (360.5, 151.9)
- added H3: MountingHole, MountingHole:MountingHole_5.3mm_M5, F.Cu at (342.6, 54.8)
- added H4: MountingHole, MountingHole:MountingHole_5.3mm_M5, F.Cu at (129.2, 54.5)
- moved J14 1.35 mm to (367.6, 146.0)
Routing:
- net Net-(J10-Pin_2): track 82.2 -> 80.5 mm
- net Net-(J14-Pin_2): track 108.1 -> 109.4 mm
- net Net-(J14-Pin_1): track 99.9 -> 101.3 mm
